File: TMC2660_Test.sch (KiCad schematic (older format))
At the start: 48 parts

Commit message: First schematic complete, netlist generated.
Parts:
- added P103: CONN_2, symbol CONN_2
- added P104: CONN_13X2, symbol CONN_13X2
- gave numbers to parts that had none: 48
Connections:
- net +12V: now also P103.1 (P1)
- net GND: now also P103.2 (PM), P104.25 (P24), P104.26 (P22)
- net MISO: now also P104.13 (P13), P104.14 (P14)
- net MOSI: now also P104.11 (P11), P104.12 (P12)
- net SCK: now also P104.15 (P15), P104.16 (P16)
- net VCC: now also P104.1 (P1), P104.2 (P2)
- net X-DIR: now also P104.5 (P5)
- net X-EN: now also P104.3 (P3)
- net X-SEL: now also P104.9 (P9)
- net X-STEP: now also P104.7 (P7)
- new net E-DIR: P104.20 (P20)
- new net E-EN: P104.18 (P18)
- new net E-SEL: P104.24 (P20)
- new net E-STEP: P104.22 (P22)
- new net Y-DIR: P104.19 (P19)
- new net Y-EN: P104.17 (P17)
- new net Y-SEL: P104.23 (P23)
- new net Y-STEP: P104.21 (P21)
- new net Z-DIR: P104.6 (P6)
- new net Z-EN: P104.4 (P4)
- new net Z-SEL: P104.10 (P10)
- new net Z-STEP: P104.8 (P8)
