File: TMC2660_Test.sch (KiCad schematic (older format))
At the start: 70 parts, among them P101 CONN_4, P102 CONN_4, P103 CONN_2, P104 CONN_13X2, P105 CONN_4, P106 CONN_4, P107 CONN_1, P108 CONN_1, P109 CONN_1, P110 CONN_1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

Commit message: Getting pretty close.
Connections:
- net E-DIR: now also P104.20 (P20); no longer P104.22 (P22)
- net E-EN: now also P104.24 (P20); no longer P104.18 (P18)
- net E-SEL: now also P104.22 (P22); no longer P104.20 (P20)
- net E-STEP: now also P104.18 (P18); no longer P104.24 (P20)
- net X-DIR: now also P104.7 (P7); no longer P104.5 (P5)
- net X-EN: now also P104.3 (P3); no longer P104.7 (P7)
- net X-SEL: now also P104.5 (P5); no longer P104.9 (P9)
- net X-STEP: now also P104.9 (P9); no longer P104.3 (P3)
- net Y-DIR: now also P104.21 (P21); no longer P104.23 (P23)
- net Y-STEP: now also P104.23 (P23); no longer P104.21 (P21)
- net Z-DIR: now also P104.6 (P6); no longer P104.4 (P4)
- net Z-EN: now also P104.10 (P10); no longer P104.8 (P8)
- net Z-SEL: now also P104.8 (P8); no longer P104.10 (P10)
- net Z-STEP: now also P104.4 (P4); no longer P104.6 (P6)
Changed lines of the file:
@@
 Text GLabel 5500 6850 0    30   Input ~ 0
 SCK
+Text GLabel 5500 6250 0    30   Input ~ 0
+X-EN
 Text GLabel 5500 6450 0    30   Input ~ 0
-X-EN
+X-DIR
+Text GLabel 5500 6550 0    30   Input ~ 0
+X-STEP
 Text GLabel 5500 6350 0    30   Input ~ 0
-X-DIR
-Text GLabel 5500 6250 0    30   Input ~ 0
-X-STEP
-Text GLabel 5500 6550 0    30   Input ~ 0
 X-SEL
 Text GLabel 5500 6950 0    30   Input ~ 0
 Y-EN
+Text GLabel 5500 7150 0    30   Input ~ 0
+Y-DIR
 Text GLabel 5500 7250 0    30   Input ~ 0
-Y-DIR
-Text GLabel 5500 7150 0    30   Input ~ 0
 Y-STEP
 Text GLabel 5500 7050 0    30   Input ~ 0
@@
 Text GLabel 6400 6850 2    30   Input ~ 0
 SCK
+Text GLabel 6400 6550 2    30   Input ~ 0
+Z-EN
+Text GLabel 6400 6350 2    30   Input ~ 0
+Z-DIR
+Text GLabel 6400 6250 2    30   Input ~ 0
+Z-STEP
 Text GLabel 6400 6450 2    30   Input ~ 0
-Z-EN
-Text GLabel 6400 6250 2    30   Input ~ 0
-Z-DIR
-Text GLabel 6400 6350 2    30   Input ~ 0
-Z-STEP
-Text GLabel 6400 6550 2    30   Input ~ 0
 Z-SEL
+Text GLabel 6400 7250 2    30   Input ~ 0
+E-EN
+Text GLabel 6400 7050 2    30   Input ~ 0
+E-DIR
 Text GLabel 6400 6950 2    30   Input ~ 0
-E-EN
+E-STEP
 Text GLabel 6400 7150 2    30   Input ~ 0
-E-DIR
-Text GLabel 6400 7250 2    30   Input ~ 0
-E-STEP
-Text GLabel 6400 7050 2    30   Input ~ 0
 E-SEL
 Wire Wire Line

Commit message: Added some notes, labels on silkscreen, and Open Source Hardware logo.
Parts:
- added M101: LOGO_OSHW, OSHW_logo_2, symbol LOGO_OSHW
Changed lines of the file:
@@
 LIBS:valves
 LIBS:trinamic
+LIBS:oshw_logo
 LIBS:TMC2660_Test-cache
 EELAYER 24 0
@@
 $EndComp
 Connection ~ 6500 4700
+$Comp
+L LOGO_OSHW M101
+U 1 1 53892EB0
+P 3650 7150
+F 0 "M101" H 3650 7300 60  0000 C CNN
+F 1 "LOGO_OSHW" H 3650 7050 60  0000 C CNN
+F 2 "OSHW_logo_2" H 3550 7200 60  0000 C CNN
+F 3 "" H 3650 7150 60  0000 C CNN
+	1    3650 7150
+	1    0    0    -1
+$EndComp
 $EndSCHEMATC

Commit message: Damn, got the input protection resistors wrong (placement and value). Now fixed.
Parts:
- R101, R102, R103, R104, R109, R110, R111, R112: value 200 -> 22
Connections:
- net at R102.2, U101.12 (SRA): now also C108.1; no longer R106.1
- net at R101.1, U101.22 (SRB): now also C107.1; no longer R105.1
- net at R101.2, U101.25 (BRB): now also R105.1; no longer C107.1
- net at R102.1, U101.9 (BRA): now also R106.1; no longer C108.1
- net at R104.2, U102.12 (SRA): now also C110.1; no longer R108.1
- net at R103.1, U102.22 (SRB): now also C109.1; no longer R107.1
- net at R103.2, U102.25 (BRB): now also R107.1; no longer C109.1
- net at R104.1, U102.9 (BRA): now also R108.1; no longer C110.1
- net at R110.2, U103.12 (SRA): now also C120.1; no longer R114.1
- net at R109.1, U103.22 (SRB): now also C119.1; no longer R113.1
- net at R109.2, U103.25 (BRB): now also R113.1; no longer C119.1
- net at R110.1, U103.9 (BRA): now also R114.1; no longer C120.1
- net at R112.2, U104.12 (SRA): now also C123.1; no longer R116.1
- net at R111.1, U104.22 (SRB): now also C122.1; no longer R115.1
- net at R111.2, U104.25 (BRB): now also R115.1; no longer C122.1
- net at R112.1, U104.9 (BRA): now also R116.1; no longer C123.1
Other:
- moved on the sheet: C107, C108, C109, C110, C119, C120, C122, C123, R105, R106, R107, R108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
Changed lines of the file:
@@
 L C C108
 U 1 1 5340332B
-P 4800 3400
-F 0 "C108" H 4800 3500 40  0000 L CNN
-F 1 "10n" H 4806 3315 40  0000 L CNN
-F 2 "" H 4838 3250 30  0000 C CNN
-F 3 "" H 4800 3400 60  0000 C CNN
-	1    4800 3400
+P 4800 2700
+F 0 "C108" H 4800 2800 40  0000 L CNN
+F 1 "10n" H 4806 2615 40  0000 L CNN
+F 2 "" H 4838 2550 30  0000 C CNN
+F 3 "" H 4800 2700 60  0000 C CNN
+	1    4800 2700
 	0    -1   -1   0
 $EndComp
@@
 L C C107
 U 1 1 53403353
-P 4800 800
-F 0 "C107" H 4800 900 40  0000 L CNN
-F 1 "10n" H 4806 715 40  0000 L CNN
-F 2 "" H 4838 650 30  0000 C CNN
-F 3 "" H 4800 800 60  0000 C CNN
-	1    4800 800
+P 4800 1500
+F 0 "C107" H 4800 1600 40  0000 L CNN
+F 1 "10n" H 4806 1415 40  0000 L CNN
+F 2 "" H 4838 1350 30  0000 C CNN
+F 3 "" H 4800 1500 60  0000 C CNN
+	1    4800 1500
 	0    -1   -1   0
 $EndComp
@@
 L R R105
 U 1 1 53403362
-P 4850 1500
-F 0 "R105" V 4930 1500 40  0000 C CNN
-F 1 "100m" V 4857 1501 40  0000 C CNN
-F 2 "" V 4780 1500 30  0000 C CNN
-F 3 "" H 4850 1500 30  0000 C CNN
-	1    4850 1500
+P 4850 800
+F 0 "R105" V 4930 800 40  0000 C CNN
+F 1 "100m" V 4857 801 40  0000 C CNN
+F 2 "" V 4780 800 30  0000 C CNN
+F 3 "" H 4850 800 30  0000 C CNN
+	1    4850 800
 	0    -1   -1   0
 $EndComp
@@
 L R R106
 U 1 1 53403371
-P 4850 2700
-F 0 "R106" V 4930 2700 40  0000 C CNN
-F 1 "100m" V 4857 2701 40  0000 C CNN
-F 2 "" V 4780 2700 30  0000 C CNN
-F 3 "" H 4850 2700 30  0000 C CNN
-	1    4850 2700
+P 4850 3400
+F 0 "R106" V 4930 3400 40  0000 C CNN
+F 1 "100m" V 4857 3401 40  0000 C CNN
+F 2 "" V 4780 3400 30  0000 C CNN
+F 3 "" H 4850 3400 30  0000 C CNN
+	1    4850 3400
 	0    -1   -1   0
 $EndComp
@@
 P 4550 1150
 F 0 "R101" V 4630 1150 40  0000 C CNN
-F 1 "200" V 4557 1151 40  0000 C CNN
+F 1 "22" V 4557 1151 40  0000 C CNN
 F 2 "" V 4480 1150 30  0000 C CNN
 F 3 "" H 4550 1150 30  0000 C CNN
@@
 P 4550 3050
 F 0 "R102" V 4630 3050 40  0000 C CNN
-F 1 "200" V 4557 3051 40  0000 C CNN
+F 1 "22" V 4557 3051 40  0000 C CNN
 F 2 "" V 4480 3050 30  0000 C CNN
 F 3 "" H 4550 3050 30  0000 C CNN
@@
 	5200 3400 5200 800
 Wire Wire Line
-	5200 3400 5000 3400
-Wire Wire Line
-	5200 800  5000 800
-Wire Wire Line
-	5100 1500 5200 1500
+	5000 1500 5200 1500
 Connection ~ 5200 1500
 Wire Wire Line
@@
 Connection ~ 5200 2500
 Wire Wire Line
-	5100 2700 5200 2700
+	5000 2700 5200 2700
 Connection ~ 5200 2700
 Wire Wire Line
@@
 L C C110
 U 1 1 5340490C
-P 4800 6500
-F 0 "C110" H 4800 6600 40  0000 L CNN
-F 1 "10n" H 4806 6415 40  0000 L CNN
-F 2 "" H 4838 6350 30  0000 C CNN
-F 3 "" H 4800 6500 60  0000 C CNN
-	1    4800 6500
+P 4800 5800
+F 0 "C110" H 4800 5900 40  0000 L CNN
+F 1 "10n" H 4806 5715 40  0000 L CNN
+F 2 "" H 4838 5650 30  0000 C CNN
+F 3 "" H 4800 5800 60  0000 C CNN
+	1    4800 5800
 	0    -1   -1   0
 $EndComp
@@
 L C C109
 U 1 1 53404918
-P 4800 3900
-F 0 "C109" H 4800 4000 40  0000 L CNN
-F 1 "10n" H 4806 3815 40  0000 L CNN
-F 2 "" H 4838 3750 30  0000 C CNN
-F 3 "" H 4800 3900 60  0000 C CNN
-	1    4800 3900
+P 4800 4600
+F 0 "C109" H 4800 4700 40  0000 L CNN
+F 1 "10n" H 4806 4515 40  0000 L CNN
+F 2 "" H 4838 4450 30  0000 C CNN
+F 3 "" H 4800 4600 60  0000 C CNN
+	1    4800 4600
 	0    -1   -1   0
 $EndComp
@@
 L R R107
 U 1 1 5340491E
-P 4850 4600
-F 0 "R107" V 4930 4600 40  0000 C CNN
-F 1 "100m" V 4857 4601 40  0000 C CNN
-F 2 "" V 4780 4600 30  0000 C CNN
-F 3 "" H 4850 4600 30  0000 C CNN
-	1    4850 4600
+P 4850 3900
+F 0 "R107" V 4930 3900 40  0000 C CNN
+F 1 "100m" V 4857 3901 40  0000 C CNN
+F 2 "" V 4780 3900 30  0000 C CNN
+F 3 "" H 4850 3900 30  0000 C CNN
+	1    4850 3900
 	0    -1   -1   0
 $EndComp
@@
 L R R108
 U 1 1 53404924
-P 4850 5800
-F 0 "R108" V 4930 5800 40  0000 C CNN
-F 1 "100m" V 4857 5801 40  0000 C CNN
-F 2 "" V 4780 5800 30  0000 C CNN
-F 3 "" H 4850 5800 30  0000 C CNN
-	1    4850 5800
+P 4850 6500
+F 0 "R108" V 4930 6500 40  0000 C CNN
+F 1 "100m" V 4857 6501 40  0000 C CNN
+F 2 "" V 4780 6500 30  0000 C CNN
+F 3 "" H 4850 6500 30  0000 C CNN
+	1    4850 6500
 	0    -1   -1   0
 $EndComp
@@
 P 4550 4250
 F 0 "R103" V 4630 4250 40  0000 C CNN
-F 1 "200" V 4557 4251 40  0000 C CNN
+F 1 "22" V 4557 4251 40  0000 C CNN
 F 2 "" V 4480 4250 30  0000 C CNN
 F 3 "" H 4550 4250 30  0000 C CNN
@@
 P 4550 6150
 F 0 "R104" V 4630 6150 40  0000 C CNN
-F 1 "200" V 4557 6151 40  0000 C CNN
+F 1 "22" V 4557 6151 40  0000 C CNN
 F 2 "" V 4480 6150 30  0000 C CNN
 F 3 "" H 4550 6150 30  0000 C CNN
@@
 	5200 6500 5200 3900
 Wire Wire Line
-	5200 6500 5000 6500
-Wire Wire Line
-	5200 3900 5000 3900
-Wire Wire Line
-	5100 4600 5200 4600
+	5000 4600 5200 4600
 Connection ~ 5200 4600
 Wire Wire Line
@@
 Connection ~ 5200 5600
 Wire Wire Line
-	5100 5800 5200 5800
+	5000 5800 5200 5800
 Connection ~ 5200 5800
 Wire Wire Line
@@
 L C C120
 U 1 1 534049F3
-P 10250 3400
-F 0 "C120" H 10250 3500 40  0000 L CNN
-F 1 "10n" H 10256 3315 40  0000 L CNN
-F 2 "" H 10288 3250 30  0000 C CNN
-F 3 "" H 10250 3400 60  0000 C CNN
-	1    10250 3400
+P 10250 2700
+F 0 "C120" H 10250 2800 40  0000 L CNN
+F 1 "10n" H 10256 2615 40  0000 L CNN
+F 2 "" H 10288 2550 30  0000 C CNN
+F 3 "" H 10250 2700 60  0000 C CNN
+	1    10250 2700
 	0    -1   -1   0
 $EndComp
@@
 L C C119
 U 1 1 534049FF
-P 10250 800
-F 0 "C119" H 10250 900 40  0000 L CNN
-F 1 "10n" H 10256 715 40  0000 L CNN
-F 2 "" H 10288 650 30  0000 C CNN
-F 3 "" H 10250 800 60  0000 C CNN
-	1    10250 800
+P 10250 1500
+F 0 "C119" H 10250 1600 40  0000 L CNN
+F 1 "10n" H 10256 1415 40  0000 L CNN
+F 2 "" H 10288 1350 30  0000 C CNN
+F 3 "" H 10250 1500 60  0000 C CNN
+	1    10250 1500
 	0    -1   -1   0
 $EndComp
@@
 L R R113
 U 1 1 53404A05
-P 10300 1500
-F 0 "R113" V 10380 1500 40  0000 C CNN
-F 1 "100m" V 10307 1501 40  0000 C CNN
-F 2 "" V 10230 1500 30  0000 C CNN
-F 3 "" H 10300 1500 30  0000 C CNN
-	1    10300 1500
+P 10300 800
+F 0 "R113" V 10380 800 40  0000 C CNN
+F 1 "100m" V 10307 801 40  0000 C CNN
+F 2 "" V 10230 800 30  0000 C CNN
+F 3 "" H 10300 800 30  0000 C CNN
+	1    10300 800
 	0    -1   -1   0
 $EndComp
@@
 L R R114
 U 1 1 53404A0B
-P 10300 2700
-F 0 "R114" V 10380 2700 40  0000 C CNN
-F 1 "100m" V 10307 2701 40  0000 C CNN
-F 2 "" V 10230 2700 30  0000 C CNN
-F 3 "" H 10300 2700 30  0000 C CNN
-	1    10300 2700
+P 10300 3400
+F 0 "R114" V 10380 3400 40  0000 C CNN
+F 1 "100m" V 10307 3401 40  0000 C CNN
+F 2 "" V 10230 3400 30  0000 C CNN
+F 3 "" H 10300 3400 30  0000 C CNN
+	1    10300 3400
 	0    -1   -1   0
 $EndComp
@@
 P 10000 1150
 F 0 "R109" V 10080 1150 40  0000 C CNN
-F 1 "200" V 10007 1151 40  0000 C CNN
+F 1 "22" V 10007 1151 40  0000 C CNN
 F 2 "" V 9930 1150 30  0000 C CNN
 F 3 "" H 10000 1150 30  0000 C CNN
@@
 P 10000 3050
 F 0 "R110" V 10080 3050 40  0000 C CNN
-F 1 "200" V 10007 3051 40  0000 C CNN
+F 1 "22" V 10007 3051 40  0000 C CNN
 F 2 "" V 9930 3050 30  0000 C CNN
 F 3 "" H 10000 3050 30  0000 C CNN
@@
 	10650 3400 10650 800
 Wire Wire Line
-	10650 3400 10450 3400
-Wire Wire Line
-	10650 800  10450 800
-Wire Wire Line
-	10550 1500 10650 1500
+	10450 1500 10650 1500
 Connection ~ 10650 1500
 Wire Wire Line
@@
 Connection ~ 10650 2500
 Wire Wire Line
-	10550 2700 10650 2700
+	10450 2700 10650 2700
 Connection ~ 10650 2700
 Wire Wire Line
@@
 L C C123
 U 1 1 53404ADA
-P 10400 6500
-F 0 "C123" H 10400 6600 40  0000 L CNN
-F 1 "10n" H 10406 6415 40  0000 L CNN
-F 2 "" H 10438 6350 30  0000 C CNN
-F 3 "" H 10400 6500 60  0000 C CNN
-	1    10400 6500
+P 10400 5800
+F 0 "C123" H 10400 5900 40  0000 L CNN
+F 1 "10n" H 10406 5715 40  0000 L CNN
+F 2 "" H 10438 5650 30  0000 C CNN
+F 3 "" H 10400 5800 60  0000 C CNN
+	1    10400 5800
 	0    -1   -1   0
 $EndComp
@@
 L C C122
 U 1 1 53404AE6
-P 10400 3900
-F 0 "C122" H 10400 4000 40  0000 L CNN
-F 1 "10n" H 10406 3815 40  0000 L CNN
-F 2 "" H 10438 3750 30  0000 C CNN
-F 3 "" H 10400 3900 60  0000 C CNN
-	1    10400 3900
+P 10400 4600
+F 0 "C122" H 10400 4700 40  0000 L CNN
+F 1 "10n" H 10406 4515 40  0000 L CNN
+F 2 "" H 10438 4450 30  0000 C CNN
+F 3 "" H 10400 4600 60  0000 C CNN
+	1    10400 4600
 	0    -1   -1   0
 $EndComp
@@
 L R R115
 U 1 1 53404AEC
-P 10450 4600
-F 0 "R115" V 10530 4600 40  0000 C CNN
-F 1 "100m" V 10457 4601 40  0000 C CNN
-F 2 "" V 10380 4600 30  0000 C CNN
-F 3 "" H 10450 4600 30  0000 C CNN
-	1    10450 4600
+P 10450 3900
+F 0 "R115" V 10530 3900 40  0000 C CNN
+F 1 "100m" V 10457 3901 40  0000 C CNN
+F 2 "" V 10380 3900 30  0000 C CNN
+F 3 "" H 10450 3900 30  0000 C CNN
+	1    10450 3900
 	0    -1   -1   0
 $EndComp
@@
 L R R116
 U 1 1 53404AF2
-P 10450 5800
-F 0 "R116" V 10530 5800 40  0000 C CNN
-F 1 "100m" V 10457 5801 40  0000 C CNN
-F 2 "" V 10380 5800 30  0000 C CNN
-F 3 "" H 10450 5800 30  0000 C CNN
-	1    10450 5800
+P 10450 6500
+F 0 "R116" V 10530 6500 40  0000 C CNN
+F 1 "100m" V 10457 6501 40  0000 C CNN
+F 2 "" V 10380 6500 30  0000 C CNN
+F 3 "" H 10450 6500 30  0000 C CNN
+	1    10450 6500
 	0    -1   -1   0
 $EndComp
@@
 P 10150 4250
 F 0 "R111" V 10230 4250 40  0000 C CNN
-F 1 "200" V 10157 4251 40  0000 C CNN
+F 1 "22" V 10157 4251 40  0000 C CNN
 F 2 "" V 10080 4250 30  0000 C CNN
 F 3 "" H 10150 4250 30  0000 C CNN
@@
 P 10150 6150
 F 0 "R112" V 10230 6150 40  0000 C CNN
-F 1 "200" V 10157 6151 40  0000 C CNN
+F 1 "22" V 10157 6151 40  0000 C CNN
 F 2 "" V 10080 6150 30  0000 C CNN
 F 3 "" H 10150 6150 30  0000 C CNN
@@
 	10800 6500 10800 3900
 Wire Wire Line
-	10800 6500 10600 6500
-Wire Wire Line
-	10800 3900 10600 3900
-Wire Wire Line
-	10700 4600 10800 4600
+	10600 4600 10800 4600
 Connection ~ 10800 4600
 Wire Wire Line
@@
 Connection ~ 10800 5600
 Wire Wire Line
-	10700 5800 10800 5800
+	10600 5800 10800 5800
 Connection ~ 10800 5800
 Wire Wire Line
@@
 	1    0    0    -1
 $EndComp
+Wire Wire Line
+	5100 6500 5200 6500
+Wire Wire Line
+	5200 3900 5100 3900
+Wire Wire Line
+	10800 3900 10700 3900
+Wire Wire Line
+	10800 6500 10700 6500
+Wire Wire Line
+	10650 800  10550 800
+Wire Wire Line
+	10550 3400 10650 3400
+Wire Wire Line
+	5200 3400 5100 3400
+Wire Wire Line
+	5200 800  5100 800
 $EndSCHEMATC
