File: TMC2660_Test.kicad_pcb (KiCad board)
At the start: 4 copper layers, 50 parts, among them P101 CONN_4, P102 CONN_4, P103 CONN_2, P104 CONN_13X2, P105 CONN_4, P106 CONN_4, U101 TMC2660, U102 TMC2660, U103 TMC2660, U104 TMC2660

Commit message: Halfway done with layout.
Parts:
- moved C102 142.0 mm to (127.5, 184.0)
- moved C106 142.0 mm to (121.0, 184.0)
- moved C117 135.7 mm to (107.4, 180.7)
- moved C118 135.7 mm to (101.0, 180.7)
- moved R103 135.7 mm to (125.4, 180.2)
- moved R104 135.7 mm to (146.5, 180.2)
- moved R111 135.7 mm to (150.7, 180.2)
- moved R112 135.7 mm to (112.8, 180.2)
- moved R115 135.7 mm to (133.9, 180.2)
- moved R116 135.7 mm to (129.6, 180.2)
- moved C104 135.7 mm to (107.4, 174.4)
- moved C109 135.7 mm to (146.1, 174.4)
- moved C110 135.7 mm to (120.3, 174.4)
- moved C123 135.7 mm to (159.0, 174.4)
- moved C124 135.7 mm to (152.6, 174.4)
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Connections:
- P104 pad 19: Y-DIR -> Y-SEL
- P104 pad 23: Y-SEL -> Y-DIR
Routing:
- net Y-SEL: track 0.00 -> 33.5 mm, vias 0 -> 1
- net VCC: track 16.0 -> 49.3 mm, vias 0 -> 1
- net MOSI: track 30.4 -> 61.8 mm, vias 1 -> 3
- net Y-EN: track 0.00 -> 30.8 mm, vias 0 -> 1
- net MISO: track 26.6 -> 55.9 mm, vias 1 -> 3
- net SCK: track 26.5 -> 48.7 mm, vias 1 -> 2
- net GND: track 13.7 -> 30.7 mm, vias 17 -> 35
- net N-0000031: track 0.00 -> 10.7 mm
- net N-0000034: track 0.00 -> 9.29 mm
- net N-000001: track 7.41 -> 16.7 mm, vias 0 -> 6
- net N-0000023: track 7.53 -> 16.5 mm, vias 0 -> 6
- net N-0000033: track 0.00 -> 7.93 mm
- net +12V: track 61.4 -> 68.6 mm, vias 3 -> 6
- net Y-STEP: track 0.00 -> 6.47 mm
- net Y-DIR: track 0.00 -> 6.44 mm
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Other:
- board outline added: 45.1 x 53.3 mm

Commit message: Adjust connector to match other side.
Connections:
- P104 pad 20: E-DIR -> E-SEL
- P104 pad 24: E-SEL -> E-DIR
- P104 pad 4: Z-EN -> Z-STEP
- P104 pad 8: Z-STEP -> Z-EN
Routing:
- net VCC: track 49.3 -> 51.8 mm
- net SCK: track 48.7 -> 51.3 mm
- net MISO: track 55.9 -> 58.4 mm
- net MOSI: track 61.8 -> 64.3 mm
Changed lines of the file:
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@@
   (general
     (links 214)
-    (no_connects 111)
-    (area 0 0 0 0)
+    (no_connects 107)
+    (area 108.915999 102.057999 154.101001 155.498001)
     (thickness 1.6)
     (drawings 4)
-    (tracks 507)
+    (tracks 511)
     (zones 0)
     (modules 50)
@@
   )
   (setup
-    (last_trace_width 0.381)
+    (last_trace_width 0.1524)
     (user_trace_width 0.381)
     (user_trace_width 0.762)
@@
     (pad 4 thru_hole circle (at -12.7 -1.27 180) (size 1.524 1.524) (drill 1.016)
       (layers *.Cu *.Mask F.SilkS)
+      (net 86 Z-STEP)
+    )
+    (pad 5 thru_hole circle (at -10.16 1.27 180) (size 1.524 1.524) (drill 1.016)
+      (layers *.Cu *.Mask F.SilkS)
+      (net 75 X-DIR)
+    )
+    (pad 6 thru_hole circle (at -10.16 -1.27 180) (size 1.524 1.524) (drill 1.016)
+      (layers *.Cu *.Mask F.SilkS)
+      (net 83 Z-DIR)
+    )
+    (pad 7 thru_hole circle (at -7.62 1.27 180) (size 1.524 1.524) (drill 1.016)
+      (layers *.Cu *.Mask F.SilkS)
+      (net 76 X-EN)
+    )
+    (pad 8 thru_hole circle (at -7.62 -1.27 180) (size 1.524 1.524) (drill 1.016)
+      (layers *.Cu *.Mask F.SilkS)
       (net 84 Z-EN)
     )
-    (pad 5 thru_hole circle (at -10.16 1.27 180) (size 1.524 1.524) (drill 1.016)
-      (layers *.Cu *.Mask F.SilkS)
-      (net 75 X-DIR)
-    )
-    (pad 6 thru_hole circle (at -10.16 -1.27 180) (size 1.524 1.524) (drill 1.016)
-      (layers *.Cu *.Mask F.SilkS)
-      (net 83 Z-DIR)
-    )
-    (pad 7 thru_hole circle (at -7.62 1.27 180) (size 1.524 1.524) (drill 1.016)
-      (layers *.Cu *.Mask F.SilkS)
-      (net 76 X-EN)
-    )
-    (pad 8 thru_hole circle (at -7.62 -1.27 180) (size 1.524 1.524) (drill 1.016)
-      (layers *.Cu *.Mask F.SilkS)
-      (net 86 Z-STEP)
-    )
     (pad 9 thru_hole circle (at -5.08 1.27 180) (size 1.524 1.524) (drill 1.016)
       (layers *.Cu *.Mask F.SilkS)
@@
     (pad 20 thru_hole circle (at 7.62 -1.27 180) (size 1.524 1.524) (drill 1.016)
       (layers *.Cu *.Mask F.SilkS)
+      (net 4 E-SEL)
+    )
+    (pad 21 thru_hole circle (at 10.16 1.27 180) (size 1.524 1.524) (drill 1.016)
+      (layers *.Cu *.Mask F.SilkS)
+      (net 82 Y-STEP)
+    )
+    (pad 22 thru_hole circle (at 10.16 -1.27 180) (size 1.524 1.524) (drill 1.016)
+      (layers *.Cu *.Mask F.SilkS)
+      (net 5 E-STEP)
+    )
+    (pad 23 thru_hole circle (at 12.7 1.27 180) (size 1.524 1.524) (drill 1.016)
+      (layers *.Cu *.Mask F.SilkS)
+      (net 79 Y-DIR)
+    )
+    (pad 24 thru_hole circle (at 12.7 -1.27 180) (size 1.524 1.524) (drill 1.016)
+      (layers *.Cu *.Mask F.SilkS)
       (net 2 E-DIR)
-    )
-    (pad 21 thru_hole circle (at 10.16 1.27 180) (size 1.524 1.524) (drill 1.016)
-      (layers *.Cu *.Mask F.SilkS)
-      (net 82 Y-STEP)
-    )
-    (pad 22 thru_hole circle (at 10.16 -1.27 180) (size 1.524 1.524) (drill 1.016)
-      (layers *.Cu *.Mask F.SilkS)
-      (net 5 E-STEP)
-    )
-    (pad 23 thru_hole circle (at 12.7 1.27 180) (size 1.524 1.524) (drill 1.016)
-      (layers *.Cu *.Mask F.SilkS)
-      (net 79 Y-DIR)
-    )
-    (pad 24 thru_hole circle (at 12.7 -1.27 180) (size 1.524 1.524) (drill 1.016)
-      (layers *.Cu *.Mask F.SilkS)
-      (net 4 E-SEL)
     )
     (pad 25 thru_hole circle (at 15.24 1.27 180) (size 1.524 1.524) (drill 1.016)
@@
   (segment (start 142.24 121.285) (end 142.24 120.142) (width 0.381) (layer F.Cu) (net 6))
   (via (at 142.24 120.142) (size 0.381) (layers F.Cu B.Cu) (net 6))
+  (segment (start 134.366 127.381) (end 134.366 129.921) (width 0.762) (layer Inner2.Cu) (net 7))
   (segment (start 125.095 118.237) (end 126.619 118.237) (width 0.381) (layer Inner1.Cu) (net 7))
   (segment (start 131.064 124.587) (end 132.461 125.984) (width 0.381) (layer F.Cu) (net 7))
@@
   (segment (start 137.16 123.444) (end 140.589 123.444) (width 0.381) (layer Inner1.Cu) (net 7))
   (segment (start 134.366 126.238) (end 137.16 123.444) (width 0.381) (layer Inner1.Cu) (net 7))
+  (segment (start 136.906 127.381) (end 136.906 129.921) (width 0.762) (layer Inner2.Cu) (net 8))
   (segment (start 131.826 118.11) (end 131.826 124.333) (width 0.381) (layer F.Cu) (net 8))
   (segment (start 131.826 124.333) (end 133.223 125.73) (width 0.381) (layer F.Cu) (net 8))
@@
   (segment (start 150.368 113.792) (end 150.368 115.189) (width 0.381) (layer F.Cu) (net 55))
   (via (at 150.368 113.792) (size 0.381) (layers F.Cu B.Cu) (net 55))
+  (segment (start 131.826 127.381) (end 131.826 129.921) (width 0.762) (layer Inner2.Cu) (net 73))
   (segment (start 130.683 125.095) (end 130.048 125.095) (width 0.381) (layer Inner1.Cu) (net 73))
   (segment (start 123.825 120.65) (end 121.793 120.65) (width 0.381) (layer Inner1.Cu) (net 73))
@@
   (segment (start 135.382 122.682) (end 140.208 122.682) (width 0.381) (layer Inner1.Cu) (net 73))
   (segment (start 131.826 126.238) (end 135.382 122.682) (width 0.381) (layer Inner1.Cu) (net 73))
+  (segment (start 149.606 127.381) (end 149.606 129.921) (width 0.762) (layer Inner2.Cu) (net 74))
   (segment (start 129.794 123.063) (end 125.603 123.063) (width 0.381) (layer F.Cu) (net 74))
   (segment (start 147.955 125.73) (end 132.461 125.73) (width 0.762) (layer Inner2.Cu) (net 74))

Commit message: Fixed a few oopsies.
Routing:
- net +12V: track 68.6 -> 74.2 mm
- net N-0000053: track 6.88 -> 9.42 mm
- net N-0000052: track 7.08 -> 9.55 mm
Changed lines of the file:
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@@
   (general
     (links 214)
-    (no_connects 107)
+    (no_connects 104)
     (area 108.915999 102.057999 154.101001 155.498001)
     (thickness 1.6)
     (drawings 4)
-    (tracks 511)
+    (tracks 516)
     (zones 0)
     (modules 50)
@@
   (layers
     (15 F.Cu signal)
-    (2 Inner2.Cu signal)
+    (2 Inner2.Cu signal hide)
     (1 Inner1.Cu signal)
     (0 B.Cu signal)
@@
   )
   (setup
-    (last_trace_width 0.1524)
+    (last_trace_width 0.381)
     (user_trace_width 0.381)
     (user_trace_width 0.762)
@@
   (gr_line (start 108.966 155.448) (end 154.051 155.448) (angle 90) (layer Edge.Cuts) (width 0.1))
   (gr_line (start 108.966 102.108) (end 108.966 155.448) (angle 90) (layer Edge.Cuts) (width 0.1))
+  (segment (start 137.16 123.825) (end 137.16 123.19) (width 0.762) (layer F.Cu) (net 1) (status C00000))
+  (segment (start 137.16 123.19) (end 135.255 121.285) (width 0.762) (layer F.Cu) (net 1) (status 400000))
+  (segment (start 139.446 123.825) (end 137.16 123.825) (width 0.762) (layer F.Cu) (net 1) (status C00000))
   (segment (start 111.506 126.238) (end 111.506 124.714) (width 1.524) (layer B.Cu) (net 1))
   (segment (start 111.506 124.714) (end 114.3635 121.8565) (width 1.524) (layer B.Cu) (net 1))
@@
   (via (at 135.255 121.285) (size 0.381) (layers F.Cu B.Cu) (net 1))
   (segment (start 136.525 117.1702) (end 135.6868 117.1702) (width 0.381) (layer F.Cu) (net 1))
+  (segment (start 135.255 120.523) (end 135.255 121.285) (width 0.381) (layer F.Cu) (net 1))
+  (segment (start 135.6868 117.1702) (end 135.255 117.602) (width 0.381) (layer F.Cu) (net 1))
   (segment (start 135.255 117.602) (end 135.255 120.523) (width 0.381) (layer F.Cu) (net 1))
-  (segment (start 135.6868 117.1702) (end 135.255 117.602) (width 0.381) (layer F.Cu) (net 1))
-  (segment (start 135.255 120.523) (end 135.255 121.285) (width 0.381) (layer F.Cu) (net 1))
   (via (at 149.479 121.285) (size 0.381) (layers F.Cu B.Cu) (net 1))
   (segment (start 149.0472 117.1702) (end 149.479 117.602) (width 0.381) (layer F.Cu) (net 1))
@@
   (segment (start 146.2405 109.855) (end 148.3995 109.855) (width 0.762) (layer F.Cu) (net 34))
   (segment (start 148.3995 109.855) (end 148.59 109.6645) (width 0.762) (layer F.Cu) (net 34))
-  (segment (start 134.112 110.2995) (end 134.5565 110.2995) (width 0.381) (layer F.Cu) (net 35))
-  (segment (start 135.3947 113.1697) (end 136.525 113.1697) (width 0.381) (layer F.Cu) (net 35))
-  (segment (start 135.255 113.03) (end 135.3947 113.1697) (width 0.381) (layer F.Cu) (net 35))
-  (segment (start 135.255 110.998) (end 135.255 113.03) (width 0.381) (layer F.Cu) (net 35))
-  (segment (start 134.5565 110.2995) (end 135.255 110.998) (width 0.381) (layer F.Cu) (net 35))
+  (segment (start 136.525 113.1697) (end 137.6553 113.1697) (width 0.381) (layer F.Cu) (net 35) (status 400000))
+  (segment (start 134.4295 110.617) (end 134.112 110.2995) (width 0.381) (layer F.Cu) (net 35) (status C00000))
+  (segment (start 137.287 110.617) (end 134.4295 110.617) (width 0.381) (layer F.Cu) (net 35) (status 800000))
+  (segment (start 137.795 111.125) (end 137.287 110.617) (width 0.381) (layer F.Cu) (net 35))
+  (segment (start 137.795 113.03) (end 137.795 111.125) (width 0.381) (layer F.Cu) (net 35))
+  (segment (start 137.6553 113.1697) (end 137.795 113.03) (width 0.381) (layer F.Cu) (net 35))
   (segment (start 134.112 110.2995) (end 132.2705 110.2995) (width 0.762) (layer F.Cu) (net 35))
   (segment (start 132.2705 110.2995) (end 131.953 109.982) (width 0.762) (layer F.Cu) (net 35))
+  (segment (start 147.955 113.1697) (end 147.0787 113.1697) (width 0.381) (layer F.Cu) (net 36) (status 400000))
+  (segment (start 149.9235 110.744) (end 150.368 110.2995) (width 0.381) (layer F.Cu) (net 36) (status C00000))
+  (segment (start 146.939 110.744) (end 149.9235 110.744) (width 0.381) (layer F.Cu) (net 36) (status 800000))
+  (segment (start 146.685 110.998) (end 146.939 110.744) (width 0.381) (layer F.Cu) (net 36))
+  (segment (start 146.685 112.776) (end 146.685 110.998) (width 0.381) (layer F.Cu) (net 36))
+  (segment (start 147.0787 113.1697) (end 146.685 112.776) (width 0.381) (layer F.Cu) (net 36))
   (segment (start 150.368 110.2995) (end 152.3365 110.2995) (width 0.762) (layer F.Cu) (net 36))
   (segment (start 152.3365 110.2995) (end 152.527 110.109) (width 0.762) (layer F.Cu) (net 36))
-  (segment (start 150.368 110.2995) (end 149.9235 110.2995) (width 0.381) (layer F.Cu) (net 36))
-  (segment (start 148.8313 113.1697) (end 147.955 113.1697) (width 0.381) (layer F.Cu) (net 36))
-  (segment (start 149.098 112.903) (end 148.8313 113.1697) (width 0.381) (layer F.Cu) (net 36))
-  (segment (start 149.098 111.125) (end 149.098 112.903) (width 0.381) (layer F.Cu) (net 36))
-  (segment (start 149.9235 110.2995) (end 149.098 111.125) (width 0.381) (layer F.Cu) (net 36))
   (segment (start 145.4404 109.855) (end 145.4404 109.0676) (width 0.381) (layer F.Cu) (net 37))
   (segment (start 149.479 104.775) (end 149.479 103.759) (width 0.381) (layer F.Cu) (net 37))

Commit message: Layout work.
Parts:
- moved C104 59.0 mm to (150.2, 133.9), turned to 180 degrees
- moved C106 54.4 mm to (141.1, 133.5)
- moved C102 51.2 mm to (135.5, 133.5)
- moved C116 48.9 mm to (105.9, 142.1)
- moved C117 42.6 mm to (108.4, 138.2)
- moved C118 42.6 mm to (102.0, 138.2)
- moved U104 3.69 mm to (120.9, 141.7)
- moved U102 2.80 mm to (142.2, 141.7)
Routing:
- net VCC: track 51.8 -> 56.2 mm
- net +12V: track 74.2 -> 76.5 mm

Commit message: Placements and most of routing done.
Parts:
- moved R107 55.8 mm to (147.7, 148.6), turned to 270 degrees
- moved C123 54.6 mm to (110.7, 148.8), turned to 270 degrees
- moved R108 50.7 mm to (136.8, 148.6), turned to 270 degrees
- moved C122 45.8 mm to (131.6, 143.4), turned to 90 degrees
- moved C124 45.5 mm to (112.4, 153.2), turned to 180 degrees
- moved R103 40.4 mm to (149.9, 148.1), turned to 90 degrees
- moved R111 39.2 mm to (128.5, 148.0), turned to 90 degrees
- moved R116 34.7 mm to (115.4, 148.6), turned to 270 degrees
- moved R104 34.3 mm to (134.6, 148.1), turned to 270 degrees
- moved R115 32.5 mm to (126.4, 148.6), turned to 270 degrees
- moved R112 32.1 mm to (113.3, 148.1), turned to 270 degrees
- moved C112 31.1 mm to (133.2, 153.2), turned to 180 degrees
- moved C110 27.8 mm to (131.6, 149.0), turned to 270 degrees
- moved C109 26.0 mm to (152.4, 149.2), turned to 270 degrees
- moved C117 18.7 mm to (126.4, 132.7), turned to 180 degrees
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Routing:
- net +12V: track 76.5 -> 122.5 mm
- net VCC: track 56.2 -> 77.8 mm
- net N-0000086: track 0.00 -> 17.1 mm, vias 0 -> 5
- net N-0000084: track 0.00 -> 16.9 mm, vias 0 -> 5
- net N-0000046: track 0.00 -> 16.8 mm, vias 0 -> 5
- net N-0000045: track 0.00 -> 16.8 mm, vias 0 -> 5
- net N-0000044: track 0.00 -> 16.6 mm, vias 0 -> 6
- net N-0000072: track 0.00 -> 16.6 mm, vias 0 -> 6
- net N-0000071: track 0.00 -> 16.5 mm, vias 0 -> 6
- net N-0000048: track 0.00 -> 16.4 mm, vias 0 -> 6
- added copper zone on B.Cu, net N-0000044
- added copper zone on F.Cu, net N-0000044
- added copper zone on B.Cu, net N-0000045
- added copper zone on F.Cu, net N-0000045
- added copper zone on B.Cu, net N-0000046
- added copper zone on F.Cu, net N-0000046
- added copper zone on B.Cu, net N-0000048
- added copper zone on F.Cu, net N-0000048
- added copper zone on B.Cu, net N-0000071
- added copper zone on F.Cu, net N-0000071
- added copper zone on B.Cu, net N-0000072
- added copper zone on F.Cu, net N-0000072
- added copper zone on B.Cu, net N-0000084
- added copper zone on F.Cu, net N-0000084
- added copper zone on B.Cu, net N-0000086
- added copper zone on F.Cu, net N-0000086

Commit message: First attempt at layout complete.
Parts:
- moved C117 8.05 mm to (118.4, 133.6), turned to 0 degrees
- moved C118 6.22 mm to (124.3, 133.7), turned to 180 degrees
- moved C102 1.02 mm to (135.5, 132.5)
- moved C106 1.02 mm to (141.1, 132.5)
Connections:
- P104 pad 22: E-STEP -> E-DIR
- P104 pad 24: E-DIR -> E-STEP
- P104 pad 4: Z-STEP -> Z-DIR
- P104 pad 6: Z-DIR -> Z-STEP
Routing:
- net MISO: track 58.4 -> 112.7 mm, vias 3 -> 5
- net GND: track 30.7 -> 81.3 mm, vias 35 -> 66
- net SCK: track 51.3 -> 100.4 mm, vias 2 -> 6
- net MOSI: track 64.3 -> 112.2 mm, vias 3 -> 5
- net +12V: track 122.5 -> 153.3 mm, vias 6 -> 12
- net Z-SEL: track 0.00 -> 26.4 mm, vias 0 -> 1
- net Z-EN: track 0.00 -> 25.8 mm, vias 0 -> 1
- net VCC: track 77.8 -> 103.5 mm, vias 1 -> 2
- net E-EN: track 0.00 -> 22.2 mm, vias 0 -> 1
- net E-SEL: track 0.00 -> 21.5 mm, vias 0 -> 1
- net Z-STEP: track 0.00 -> 12.1 mm
- net Z-DIR: track 0.00 -> 11.4 mm
- net E-DIR: track 0.00 -> 10.4 mm
- net N-0000074: track 0.00 -> 9.75 mm
- net N-0000073: track 0.00 -> 9.48 mm
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
Commit message: Cleanup, fix an oopsie.
Routing:
- net GND: track 81.3 -> 60.1 mm
- net N-0000047: track 8.11 -> 10.5 mm
- net (no net): track 0.89 -> 0.00 mm
