File: TMC2660_Test.kicad_pcb (KiCad board)
At the start: 2 copper layers, 77.7 x 49.9 mm, 70 parts, among them P101 CONN_4, P102 CONN_4, P103 CONN_2, P104 CONN_13X2, P105 CONN_4, P106 CONN_4, P107 CONN_1, P108 CONN_1, P109 CONN_1, P110 CONN_1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

Commit message: Getting pretty close.
Parts:
- moved C118 0.35 mm to (205.8, 129.9)
Connections:
- P104 pad 10: Z-SEL -> Z-EN
- P104 pad 18: E-EN -> E-STEP
- P104 pad 20: E-SEL -> E-DIR
- P104 pad 21: Y-STEP -> Y-DIR
- P104 pad 22: E-DIR -> E-SEL
- P104 pad 23: Y-DIR -> Y-STEP
- P104 pad 24: E-STEP -> E-EN
- P104 pad 3: X-STEP -> X-EN
- P104 pad 4: Z-DIR -> Z-STEP
- P104 pad 5: X-DIR -> X-SEL
- P104 pad 6: Z-STEP -> Z-DIR
- P104 pad 7: X-EN -> X-DIR
- P104 pad 8: Z-EN -> Z-SEL
- P104 pad 9: X-SEL -> X-STEP
Routing:
- net VCC: track 50.4 -> 196.9 mm, vias 0 -> 7
- net SCK: track 29.4 -> 96.1 mm, vias 0 -> 5
- net MISO: track 54.1 -> 109.2 mm, vias 2 -> 5
- net MOSI: track 51.5 -> 102.5 mm, vias 2 -> 3
- net Y-DIR: track 0.00 -> 33.9 mm, vias 0 -> 2
- net E-STEP: track 0.00 -> 33.1 mm, vias 0 -> 2
- net Y-STEP: track 0.00 -> 32.4 mm, vias 0 -> 2
- net E-DIR: track 0.00 -> 32.0 mm, vias 0 -> 2
- net Z-STEP: track 0.00 -> 31.9 mm, vias 0 -> 1
- net Z-DIR: track 0.00 -> 30.0 mm, vias 0 -> 1
- net X-DIR: track 0.00 -> 29.8 mm, vias 0 -> 2
- net X-STEP: track 0.00 -> 29.3 mm, vias 0 -> 1
- net Y-EN: track 0.00 -> 24.4 mm
- net Y-SEL: track 0.00 -> 22.2 mm
- net E-SEL: track 0.00 -> 22.2 mm
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- added copper zone on F.Cu, net N-0000018
- removed copper zone on F.Cu, net N-0000013
- removed copper zone on F.Cu, net N-0000028
